Commit message: Update RRT as expert planner and fix robot urdf frame

File: env/models/tm5_900/robotiq_85.urdf (robot description, URDF)
Before this commit: robot tm5_900, 21 links, 20 joints
Links:
- removed link arm_1_link
- removed link arm_2_link
- removed link base_link
- removed link camera_link
- removed link flange_link
- removed link shoulder_1_link
- removed link wrist_1_link
- removed link wrist_2_link
- removed link wrist_3_link
- link left_inner_finger_pad: mass 0.02 -> 1.
- link right_inner_finger_pad: mass 0.02 -> 1
Joints:
- removed joint base-base_link
- removed joint elbow_joint
- removed joint flange_fixed_joint
- removed joint hand_camera_joint
- removed joint shoulder_1_joint
- removed joint shoulder_2_joint
- removed joint wrist_1_joint
- removed joint wrist_2_joint
- removed joint wrist_3_joint
- joint finger_joint: limit lower=0 upper=0.8 effort=1000 velocity=2.0 -> (none); type revolute -> fixed
- joint gripper_hand_joint: parent flange_link -> base
- joint left_inner_finger_joint: limit lower=-0.8757 upper=0 effort=1000 velocity=2.0 -> (none); type revolute -> fixed
- joint left_inner_knuckle_joint: limit lower=0 upper=0.8757 effort=1000 velocity=2.0 -> (none); type revolute -> fixed
- joint right_inner_finger_joint: limit lower=-0.8757 upper=0 effort=1000 velocity=2.0 -> (none); type revolute -> fixed
- joint right_inner_knuckle_joint: limit lower=0 upper=0.8757 effort=1000 velocity=2.0 -> (none); type revolute -> fixed
- joint right_outer_knuckle_joint: limit lower=0 upper=0.81 effort=1000 velocity=2.0 -> (none); type revolute -> fixed
