Commit message: Add pybullet support for acronym dataset

File: env/models/tm5_900/tm5_900_with_gripper.urdf (robot description, URDF)
Before this commit: robot tm5_900, 21 links, 20 joints
Joints:
- joint wrist_1_joint: limit lower=-3.14159 upper=3.14159 effort=150.0 velocity=3.15 -> lower=-3.14159 upper=3.14159 effort=30.0 velocity=3.15
- joint wrist_2_joint: limit lower=-3.14159 upper=3.14159 effort=150.0 velocity=3.15 -> lower=-3.14159 upper=3.14159 effort=30.0 velocity=3.15
- joint wrist_3_joint: limit lower=-4.712384999999999 upper=4.712384999999999 effort=150.0 velocity=3.15 -> lower=-4.712384999999999 upper=4.712384999999999 effort=30.0 velocity=3.15
